File: CHARGING_LINE_SCHEMATIC.sch (KiCad schematic (older format))
At the start: 30 parts, among them J1 Conn_01x06_Male, J2 Screw_Terminal_01x02, J3 Conn_01x03_Male, J4 Conn_01x03_Male, Q1 AON7407, Q2 SI7615CDN-T1-GE3 d.n.p., Q3 SIA427DJ-T1-GE3 d.n.p., SW1 RESET, SW2 HW_BUTTON, U1 AD8551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

Commit message: snapshot as of 11.10.20
Parts:
- removed C1: 100n, Capacitor_SMD:C_0805_2012Metric_Pad1.15x1.40mm_HandSolder, symbol Device:C_Small
- removed Q2: SI7615CDN-T1-GE3 d.n.p., Package_SO:Vishay_PowerPAK_1212-8_Single, symbol Device:Q_PMOS_DGS
- removed Q3: SIA427DJ-T1-GE3 d.n.p., Package_TO_SOT_SMD:Vishay_PowerPAK_SC70-6L_Single, symbol pmos_ppak:Q_PMOS_DGS
- removed U2: alt opamp - dnp, Package_TO_SOT_SMD:SOT-23-5_HandSoldering, symbol pmos_ppak:Opamp_single_sot-23-5
- BT1: value Battery_Cell -> LiIon_Cell
- Q1: value AON7407 -> AON7423
- R5: value 9k -> 100K
- R6: value 1k -> 10K
- Rs1: value 83m 0.5% -> 80m 1%
Connections:
- no-connect marks 1 -> 0
Other:
- note removed: "0.5%, low tempco"
- moved on the sheet: R5, R6, R9, Rs1
